File: bosch_shuttle_carrier.kicad_pcb (KiCad board)
At the start: 2 copper layers, 27.4 x 21.3 mm, 8 parts, among them J1 VddIO, P1 Raspberry Pi Connector, P2 Qwiic Connector, P3 Conn_01x07, P4 Conn_01x09

Commit message: Add schematics v1.0 board
Routing:
- net VDD: track 50.5 -> 48.0 mm
