File: bosch_shuttle_carrier.kicad_sch (KiCad schematic)
At the start: 8 parts, among them J1 VDDIO, P1 Raspberry Pi Connector, P2 Qwiic Connector, P3 Conn_01x07, P4 Conn_01x09

Commit message: Add schematics v1.0 board
Other:
- moved on the sheet: J1, JP1, P1, P2, P3, P4, R1, R2
